File: electronic/electronic.kicad_sch (KiCad schematic)
At the start: 55 parts, among them J1 POWER SUPLY, J10 MOT_W_ENCODER, J11 Conn_01x02, J12 Conn_01x02, J13 Conn_01x02, J14 DRVO01, J15 DRVO01, J16 Screw_Terminal_01x03, J17 Conn_01x04, J18 Conn_01x02, J19 Conn_01x02, J2 MOT_W_ENCODER, J20 Conn_01x02, J21 DRVO01, J22 Screw_Terminal_01x03, J23 DRVO01, J24 Conn_01x04, J25 Conn_01x05, J26 Conn_01x04, J27 Conn_01x04, J28 Conn_01x05, J3 M01, J4 ENC01, J5 M01, J6 ENC01, J7 MOT_W_ENCODER, J8 M01, J9 ENC01, U1 ESP32-S3-DevKitC, U2 L298N, U3 LM78M05_TO252, U4 L298N, U5 LM78M05_TO252

Commit message: chore: pcd made
Parts:
- added D19, D20, D21, D22: LED, LED_SMD:LED_Yuji_5730, symbol Device:LED
- added R3, R4, R5, R6: 330, Resistor_SMD:R_1206_3216Metric, symbol Device:R_US
- J1: footprint (none) -> Connector_BarrelJack:BarrelJack_GCT_DCJ200-10-A_Horizontal; symbol Connector_Generic:Conn_01x02 -> Connector_Generic:Conn_01x03
- J10: value MOT_W_ENCODER -> MOT_W_ENCODER03
- J2: value MOT_W_ENCODER -> MOT_W_ENCODER01
- J25, J28: footprint (none) -> Connector_JST:JST_XH_B5B-XH-A_1x05_P2.50mm_Vertical
- J26, J27, J4: footprint (none) -> Connector_JST:JST_XH_B4B-XH-A_1x04_P2.50mm_Vertical
- J3: footprint (none) -> Connector_JST:JST_XH_B2B-XH-A_1x02_P2.50mm_Vertical
- J5: value M01 -> M02; footprint (none) -> Connector_JST:JST_XH_B2B-XH-A_1x02_P2.50mm_Vertical
- J6: value ENC01 -> ENC02; footprint (none) -> Connector_JST:JST_XH_B4B-XH-A_1x04_P2.50mm_Vertical
- J7: value MOT_W_ENCODER -> MOT_W_ENCODER02
- J8: value M01 -> M03; footprint (none) -> Connector_JST:JST_XH_B2B-XH-A_1x02_P2.50mm_Vertical
- J9: value ENC01 -> ENC03; footprint (none) -> Connector_JST:JST_XH_B4B-XH-A_1x04_P2.50mm_Vertical
- U2, U4: now in the parts list
Connections:
- net DRVI101: now also U1.12 (GPIO8/ADC1_CH7)
- net DRVI102: now also U1.41 (GPIO1/ADC1_CH0)
- net DRVI201: now also U1.13 (GPIO3/ADC1_CH2)
- net DRVI202: now also U1.40 (GPIO2/ADC1_CH1)
- net DRVI301: now also U1.15 (GPIO9/ADC1_CH8)
- net DRVI401: now also U1.16 (GPIO10/ADC1_CH9)
- net Earth: now also R3.2, R4.2, R5.2, R6.2
- net L_ENC_1: now reaches U1.17 (GPIO11/ADC2_CH0)
- net L_ENC_1: now also D19.2 (A)
- net L_ENC_2: now reaches U1.18 (GPIO12/ADC2_CH1)
- net L_ENC_2: now also D20.2 (A)
- net L_ENC_3: now reaches U1.19 (GPIO13/ADC2_CH2)
- net L_ENC_3: now also D21.2 (A)
- net L_ROS: now reaches U1.20 (GPIO14/ADC2_CH3)
- net L_ROS: now also D22.2 (A)
- new net: D21.1 (K), R5.1
- new net: D20.1 (K), R4.1
- new net: D22.1 (K), R6.1
- new net: D19.1 (K), R3.1
- no-connect marks 33 -> 24
Other:
- note added: "LEDS"
- moved on the sheet: U1

Commit message: chore: PCB updated
Connections:
- net DRVI102: now also U1.10 (GPIO17/ADC2_CH6); no longer U1.41 (GPIO1/ADC1_CH0)
- net DRVI202: now also U1.11 (GPIO18/ADC2_CH7); no longer U1.40 (GPIO2/ADC1_CH1)
Changed lines of the file:
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@@
 	)
 	(no_connect
+		(at 240.03 88.9)
+	)
+	(no_connect
 		(at 189.23 86.36)
 	)
@@
 	)
 	(no_connect
-		(at 240.03 121.92)
+		(at 240.03 142.24)
 	)
 	(no_connect
-		(at 240.03 142.24)
+		(at 240.03 86.36)
 	)
 	(no_connect
@@
 	)
 	(no_connect
-		(at 240.03 124.46)
-	)
-	(no_connect
 		(at 240.03 66.04)
 	)
@@
 		)
 	)
-	(global_label "DRVI202"
-		(shape input)
-		(at 240.03 88.9 0)
-		(fields_autoplaced yes)
-		(effects
-			(font
-				(size 1.27 1.27)
-			)
-			(justify left)
-		)
-		(property "Intersheetrefs" "${INTERSHEET_REFS}"
-			(at 250.8771 88.9 0)
-			(effects
-				(font
-					(size 1.27 1.27)
-				)
-				(justify left)
-				(hide yes)
-			)
-		)
-	)
 	(global_label "DRVO302"
 		(shape input)
@@
 		)
 	)
+	(global_label "DRVI202"
+		(shape input)
+		(at 240.03 124.46 0)
+		(fields_autoplaced yes)
+		(effects
+			(font
+				(size 1.27 1.27)
+			)
+			(justify left)
+		)
+		(property "Intersheetrefs" "${INTERSHEET_REFS}"
+			(at 250.8771 124.46 0)
+			(effects
+				(font
+					(size 1.27 1.27)
+				)
+				(justify left)
+				(hide yes)
+			)
+		)
+	)
 	(global_label "PH_A01"
 		(shape input)
@@
 		)
 	)
-	(global_label "DRVI102"
-		(shape input)
-		(at 240.03 86.36 0)
-		(fields_autoplaced yes)
-		(effects
-			(font
-				(size 1.27 1.27)
-			)
-			(justify left)
-		)
-		(property "Intersheetrefs" "${INTERSHEET_REFS}"
-			(at 250.8771 86.36 0)
-			(effects
-				(font
-					(size 1.27 1.27)
-				)
-				(justify left)
-				(hide yes)
-			)
-		)
-	)
 	(global_label "DRVI101"
 		(shape input)
@@
 				(hide yes)
 			)
+		)
+	)
+	(global_label "DRVI102"
+		(shape input)
+		(at 240.03 121.92 0)
+		(fields_autoplaced yes)
+		(effects
+			(font
+				(size 1.27 1.27)
+			)
+			(justify left)
+		)
+		(property "Intersheetrefs" "${INTERSHEET_REFS}"
+			(at 250.8771 121.92 0)
+			(effects
+				(font
+					(size 1.27 1.27)
+				)
+				(justify left)
+				(hide yes)
+			)

Commit message: chore: PCB updated
Parts:
- added J29, J30: Screw_Terminal_01x03, Connector_JST:JST_XH_B3B-XH-A_1x03_P2.50mm_Vertical, symbol Connector_Generic:Conn_01x03
Connections:
- net +12V: now also J29.1 (Pin_1), J30.1 (Pin_1)
- net +5V: now also J29.3 (Pin_3), J30.3 (Pin_3)
- net Earth: now also J29.2 (Pin_2), J30.2 (Pin_2)
Other:
- moved on the sheet: J25, J26, J27, J28

Commit message: chore: gerbar and images added
Parts:
- R3, R4, R5, R6: value 330 -> 220
Changed lines of the file:
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@@
 			)
 		)
-		(property "Value" "330"
+		(property "Value" "220"
 			(at 229.8699 39.37 0)
 			(effects
@@
 			)
 		)
-		(property "Value" "330"
+		(property "Value" "220"
 			(at 265.4299 26.67 0)
 			(effects
@@
 			)
 		)
-		(property "Value" "330"
+		(property "Value" "220"
 			(at 229.8699 26.67 0)
 			(effects
@@
 			)
 		)
-		(property "Value" "330"
+		(property "Value" "220"
 			(at 265.4299 39.37 0)
 			(effects
