File: electronic/electronic.kicad_pcb (KiCad board)
At the start: 2 copper layers, 68.5 x 75 mm, 24 parts, among them J1 POWER SUPLY, J25 Conn_01x05, J26 Conn_01x04, J27 Conn_01x04, J28 Conn_01x05, J29 Screw_Terminal_01x03, J3 M01, J30 Screw_Terminal_01x03, J4 ENC01, J5 M02, J6 ENC02, J8 M03, J9 ENC03, U1 ESP32-S3-DevKitC

Commit message: chore: PCB updated
Parts:
- R3, R4, R5, R6: value 330 -> 220
Routing:
- net +12V: track 42.4 -> 43.3 mm
Changed lines of the file:
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@@
 			)
 		)
-		(property "Value" "330"
+		(property "Value" "220"
 			(at 0 1.82 90)
 			(layer "F.Fab")
@@
 			)
 		)
-		(property "Value" "330"
+		(property "Value" "220"
 			(at 0 1.82 90)
 			(layer "F.Fab")
@@
 			)
 		)
-		(property "Value" "330"
+		(property "Value" "220"
 			(at 0 1.82 90)
 			(layer "F.Fab")
@@
 			)
 		)
-		(property "Value" "330"
+		(property "Value" "220"
 			(at 0 1.82 90)
 			(layer "F.Fab")
@@
 		(tags "mounting hole 3.2mm m3 iso7380")
 		(property "Reference" "REF**"
-			(at 0 -3.85 0)
+			(at 0 4.5 0)
 			(layer "F.SilkS")
 			(effects
@@
 		(start 63.50272 77.64)
 		(end 65.5 79.63728)
-		(width 0.2)
+		(width 0.6)
 		(layer "F.Cu")
 		(net 9)
@@
 		(start 65.5 79.63728)
 		(end 69 79.63728)
-		(width 0.2)
+		(width 0.6)
 		(layer "F.Cu")
 		(net 9)
@@
 		(start 59.86 77.64)
 		(end 63.50272 77.64)
-		(width 0.2)
+		(width 0.6)
 		(layer "F.Cu")
 		(net 9)
 	)
 	(segment
-		(start 68 46)
-		(end 68 72.33728)
+		(start 68 72.33728)
+		(end 69 73.33728)
 		(width 0.2)
 		(layer "F.Cu")
@@
 	)
 	(segment
-		(start 68 34)
-		(end 70.067868 36.067868)
-		(width 0.2)
+		(start 70.5 35)
+		(end 69.5 34)
+		(width 0.6)
 		(layer "F.Cu")
 		(net 10)
 	)
 	(segment
-		(start 70.067868 45.500859)
-		(end 69.568727 46)
-		(width 0.2)
+		(start 68 46)
+		(end 69 46)
+		(width 0.6)
 		(layer "F.Cu")
 		(net 10)
 	)
 	(segment
-		(start 70.067868 36.067868)
-		(end 70.067868 45.500859)
-		(width 0.2)
+		(start 69 46)
+		(end 70.5 44.5)
+		(width 0.6)
 		(layer "F.Cu")
 		(net 10)
 	)
 	(segment
-		(start 69.568727 46)
-		(end 68 46)
-		(width 0.2)
+		(start 69.5 34)
+		(end 68 34)
+		(width 0.6)
 		(layer "F.Cu")
 		(net 10)
 	)
 	(segment
-		(start 68 72.33728)
-		(end 69 73.33728)
-		(width 0.2)
+		(start 70.5 44.5)
+		(end 70.5 35)
+		(width 0.6)
+		(layer "F.Cu")
+		(net 10)
+	)
+	(segment
+		(start 68 46)
+		(end 68 72.33728)
+		(width 0.6)
 		(layer "F.Cu")
 		(net 10)
@@
 		(layer "F.Cu")
 		(hatch edge 0.5)
-		(connect_pads
-			(clearance 0.5)
+		(connect_pads yes
+			(clearance 0.4)
 		)
-		(min_thickness 0.25)
+		(min_thickness 0.1)
 		(filled_areas_thickness no)
 		(fill yes
-			(thermal_gap 0.5)
-			(thermal_bridge_width 0.5)
+			(thermal_gap 0.6)
+			(thermal_bridge_width 1)
+			(smoothing fillet)
+			(radius 0.5)
 		)
 		(polygon
