Commit message: chore(carobot): rename *_*.STL files to *.STL and add launcher for display the project in rviz2

File: ros-ws/src/carobot/urdf/model.urdf (robot description, URDF)
Before this commit: robot CartesianRobot, 4 links, 3 joints
Links:
- added link world
- link Link_Base: geometry collision mesh filename=file:///home/akey/Unix/projects/design/ros-ws/src/carobot/u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; visual mesh filename=file:///home/akey/Unix/projects/design/ros-ws/src/carobot/u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
- link Link_X: geometry collision mesh filename=file:///home/akey/Unix/projects/design/ros-ws/src/carobot/u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; visual mesh filename=file:///home/akey/Unix/projects/design/ros-ws/src/carobot/u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
- link Link_Y: geometry collision mesh filename=file:///home/akey/Unix/projects/design/ros-ws/src/carobot/u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; visual mesh filename=file:///home/akey/Unix/projects/design/ros-ws/src/carobot/u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
- link Link_Z: geometry collision mesh filename=file:///home/akey/Unix/projects/design/ros-ws/src/carobot/u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; visual mesh filename=file:///home/akey/Unix/projects/design/ros-ws/src/carobot/u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
Joints:
- added joint world_to_base: type fixed, parent world, child Link_Base, origin xyz=0 0 0 rpy=0 0 0

Commit message: fix(model.urdf): coorect position and limit of joints and links in the model

File: ros-ws/src/carobot/urdf/model.urdf (robot description, URDF)
Before this commit: robot CartesianRobot, 5 links, 4 joints
Joints:
- joint J1: limit lower=0 upper=0.5 effort=1000 velocity=1 -> lower=-0.186 upper=0 effort=1000 velocity=1; origin xyz=-0.017414 0 0 rpy=1.5708 0 1.5708 -> xyz=0.06 0.104 0.3215 rpy=1.5708 0 1.5708
- joint J2: limit lower=0 upper=0.5 effort=1000 velocity=0 -> lower=-0.195 upper=0 effort=1000 velocity=0; origin xyz=-0.08694 0 0.018911 rpy=0 0 0 -> xyz=-0.0335 0.0395 0.0005 rpy=0 0 0
- joint J3: limit lower=0 upper=0.5 effort=1000 velocity=0 -> lower=0 upper=0.224 effort=1000 velocity=0; origin xyz=0.028485 0.10235 0 rpy=0 0 0 -> xyz=0.0006 0 0.0295 rpy=0 0 0

Commit message: Revert "fix(model.urdf): coorect position and limit of joints and links in the model"
This reverts commit 3ffb0695d2ab54cb5759cbb24cd0175b31b29e9f.

File: ros-ws/src/carobot/urdf/model.urdf (robot description, URDF)
Before this commit: robot CartesianRobot, 5 links, 4 joints
Joints:
- joint J1: limit lower=-0.186 upper=0 effort=1000 velocity=1 -> lower=0 upper=0.5 effort=1000 velocity=1; origin xyz=0.06 0.104 0.3215 rpy=1.5708 0 1.5708 -> xyz=-0.017414 0 0 rpy=1.5708 0 1.5708
- joint J2: limit lower=-0.195 upper=0 effort=1000 velocity=0 -> lower=0 upper=0.5 effort=1000 velocity=0; origin xyz=-0.0335 0.0395 0.0005 rpy=0 0 0 -> xyz=-0.08694 0 0.018911 rpy=0 0 0
- joint J3: limit lower=0 upper=0.224 effort=1000 velocity=0 -> lower=0 upper=0.5 effort=1000 velocity=0; origin xyz=0.0006 0 0.0295 rpy=0 0 0 -> xyz=0.028485 0.10235 0 rpy=0 0 0

Commit message: fix(model.urdf): correct some definitions

File: ros-ws/src/carobot/urdf/model.urdf (robot description, URDF)
Before this commit: robot CartesianRobot, 5 links, 4 joints
Links:
- link Link_X: mass 8.67596987352087 -> 0.867596987352087
- link Link_Y: mass 8.67596987352087 -> 0.0867596987352087
- link Link_Z: mass 8.67596987352087 -> 0.0867596987352087
Joints:
- joint J1: limit lower=-0.186 upper=0 effort=1000 velocity=1 -> lower=-0.186 upper=0 effort=1000 velocity=100
- joint J2: limit lower=-0.195 upper=0 effort=1000 velocity=0 -> lower=-0.184 upper=0 effort=1000 velocity=10
- joint J3: limit lower=0 upper=0.224 effort=1000 velocity=0 -> lower=0 upper=0.224 effort=1000 velocity=100

Commit message: chore(model.urdf): test pid configurations

File: ros-ws/src/carobot/urdf/model.urdf (robot description, URDF)
Before this commit: robot CartesianRobot, 5 links, 4 joints
Links:
- link Link_Y: mass 0.0867596987352087 -> 0.04867596987352087
Joints:
- joint J1: limit lower=-0.186 upper=0 effort=1000 velocity=100 -> lower=-0.186 upper=0 effort=1000 velocity=2
- joint J2: limit lower=-0.184 upper=0 effort=1000 velocity=10 -> lower=-0.184 upper=0 effort=1000 velocity=2
- joint J3: limit lower=0 upper=0.224 effort=1000 velocity=100 -> lower=0 upper=0.224 effort=5000 velocity=2

Commit message: chore(ros-ws): edit model.urdf

File: ros-ws/src/carobot/urdf/model.urdf (robot description, URDF)
Before this commit: robot CartesianRobot, 5 links, 4 joints
Links:
- link Link_Base: mass 8.67596987352087 -> 8.09
- link Link_X: mass 0.867596987352087 -> 0.32
- link Link_Y: mass 0.04867596987352087 -> 0.21

Commit message: refactor(ros-ws): update joint_state publisher based in data of gz sim

File: ros-ws/src/carobot/urdf/model.urdf (robot description, URDF)
Before this commit: robot CartesianRobot, 5 links, 4 joints
Links:
- removed link Link_Base
- removed link Link_X
- removed link Link_Y
- removed link Link_Z
- removed link world
- added link base_link, mass 8.09; collision mesh filename=file:///home/akey/Unix/projects/design/ros-ws/src/carobot/u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; visual mesh filename=file:///home/akey/Unix/projects/design/ros-ws/src/carobot/u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
- added link prismatic_0, mass 0.32; collision mesh filename=file:///home/akey/Unix/projects/design/ros-ws/src/carobot/u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; visual mesh filename=file:///home/akey/Unix/projects/design/ros-ws/src/carobot/u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
- added link prismatic_1, mass 0.0867596987352087; collision mesh filename=file:///home/akey/Unix/projects/design/ros-ws/src/carobot/u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; visual mesh filename=file:///home/akey/Unix/projects/design/ros-ws/src/carobot/u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
- added link prismatic_2, mass 0.21; collision mesh filename=file:///home/akey/Unix/projects/design/ros-ws/src/carobot/u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; visual mesh filename=file:///home/akey/Unix/projects/design/ros-ws/src/carobot/u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
Joints:
- removed joint J1
- removed joint J2
- removed joint J3
- removed joint world_to_base
- added joint prismatic_0_joint: type prismatic, parent base_link, child prismatic_0, origin xyz=0.06 0.104 0.3215 rpy=1.5708 0 1.5708, axis 0 0 1, limit lower=-0.186 upper=0 effort=5 velocity=2
- added joint prismatic_1_joint: type prismatic, parent prismatic_0, child prismatic_1, origin xyz=-0.0335 0.0395 0.0005 rpy=0 0 0, axis 1 0 0, limit lower=-0.184 upper=0 effort=5 velocity=2
- added joint prismatic_2_joint: type prismatic, parent prismatic_1, child prismatic_2, origin xyz=0.0006 0 0.0295 rpy=0 0 0, axis 0 1 0, limit lower=0 upper=0.224 effort=5 velocity=2

Commit message: refactor(ros-ws): change the filename attrib in urdf to use relative directory based on the project

File: ros-ws/src/carobot/urdf/model.urdf (robot description, URDF)
Before this commit: robot CartesianRobot, 4 links, 3 joints
Links:
- link base_link: geometry collision mesh filename=file://$(find carobot)/urdf/meshes/Base.STL; visual mesh filename=file://$(find carobot)/urdf/meshes/Base.STL
- link prismatic_0: geometry collision mesh filename=file://$(find carobot)/urdf/meshes/X.STL; visual mesh filename=file://$(find carobot)/urdf/meshes/X.STL
- link prismatic_1: geometry collision mesh filename=file://$(find carobot)/urdf/meshes/Z.STL; visual mesh filename=file://$(find carobot)/urdf/meshes/Z.STL
- link prismatic_2: geometry collision mesh filename=file://$(find carobot)/urdf/meshes/Y.STL; visual mesh filename=file://$(find carobot)/urdf/meshes/Y.STL

Commit message: fix(model.urdf): update meshes and limits for new stl files

File: ros-ws/src/carobot/urdf/model.urdf (robot description, URDF)
Before this commit: robot CartesianRobot, 4 links, 3 joints
Joints:
- joint prismatic_0_joint: limit lower=-0.186 upper=0 effort=5 velocity=2 -> lower=-0.104 upper=0.09 effort=5 velocity=2; origin xyz=0.06 0.104 0.3215 rpy=1.5708 0 1.5708 -> xyz=0.1135 0 0.3215 rpy=1.5708 0 0
- joint prismatic_1_joint: limit lower=-0.184 upper=0 effort=5 velocity=2 -> lower=-0.0865 upper=0.0865 effort=5 velocity=2; origin xyz=-0.0335 0.0395 0.0005 rpy=0 0 0 -> xyz=-0.1628 0.0365 0.0005 rpy=0 0 0
- joint prismatic_2_joint: limit lower=0 upper=0.224 effort=5 velocity=2 -> lower=-0.0889 upper=0.0889 effort=5 velocity=2; origin xyz=0.0006 0 0.0295 rpy=0 0 0 -> xyz=0.037 0.0345 0.026 rpy=0 0 0

Commit message: fix(carobot): update model

File: ros-ws/src/carobot/urdf/model.urdf (robot description, URDF)
Before this commit: robot CartesianRobot, 4 links, 3 joints
Links:
- link base_link: mass 8.09 -> 8.22
- link prismatic_0: mass 0.32 -> 0.398
- link prismatic_1: mass 0.0867596987352087 -> 0.08073
- link prismatic_2: mass 0.21 -> 0.30612

Commit message: refactor(robot): restructures ROS2

File: ros-ws/src/carobot/urdf/model.urdf (robot description, URDF)
Before this commit: robot CartesianRobot, 4 links, 3 joints
Links:
- link prismatic_2: mass 0.30612 -> .030612
Joints:
- joint prismatic_0_joint: axis 0 0 1 -> 0 0 -1; limit lower=-0.104 upper=0.09 effort=5 velocity=2 -> lower=-0.104 upper=0.09 effort=5e3 velocity=20
- joint prismatic_1_joint: limit lower=-0.0865 upper=0.0865 effort=5 velocity=2 -> lower=-0.0865 upper=0.0865 effort=5e3 velocity=20
- joint prismatic_2_joint: axis 0 1 0 -> 0 -1 0; limit lower=-0.0889 upper=0.0889 effort=5 velocity=2 -> lower=-0.0889 upper=0.0889 effort=5e3 velocity=20
